File: kicad/lora_adapter/lora_adapter.kicad_sch (KiCad schematic)
At the start: 3 parts, among them J1 Conn_02x08_Counter_Clockwise, J2 Conn_Coaxial, U1 RFM9X

Commit message: lora adapter updated
Parts:
- removed J1: Conn_02x08_Counter_Clockwise, Connector_PinHeader_2.54mm:PinHeader_2x08_P2.54mm_Vertical, symbol Connector_Generic:Conn_02x08_Counter_Clockwise
- added J1: Conn_02x08_Odd_Even, Connector_PinHeader_2.54mm:PinHeader_2x08_P2.54mm_Vertical, symbol Connector_Generic:Conn_02x08_Odd_Even
Connections:
- net +3.3V: now also J1.13 (Pin_13), J1.15 (Pin_15)
- net DIO0: now also J1.11 (Pin_11)
- net GND: now also J1.14 (Pin_14), J1.16 (Pin_16)
- net MISO: now also J1.6 (Pin_6)
- net MOSI: now also J1.7 (Pin_7)
- net NSS: now also J1.5 (Pin_5)
- net RST: now also J1.9 (Pin_9)
- net SCK: now also J1.12 (Pin_12)
Changed lines of the file:
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@@
     )
   )
-  (symbol (lib_id "Connector_Generic:Conn_02x08_Counter_Clockwise") (at 160.02 88.9 0) (unit 1)
+  (symbol (lib_id "Connector_Generic:Conn_02x08_Odd_Even") (at 160.02 88.9 0) (unit 1)
     (in_bom yes) (on_board yes) (dnp no) (fields_autoplaced)
     (property "Reference" "J1" (at 161.29 74.93 0)
       (effects (font (size 1.27 1.27)))
     )
-    (property "Value" "Conn_02x08_Counter_Clockwise" (at 161.29 77.47 0)
+    (property "Value" "Conn_02x08_Odd_Even" (at 161.29 77.47 0)
       (effects (font (size 1.27 1.27)))
     )
